File: pcb/map-and-egt-daughterboard/map-and-egt-daughterboard.kicad_pcb (KiCad board)
At the start: 2 copper layers, 46 x 46 mm, 54 parts, among them J1 B4B-PH-K-S(LF)(SN), J2 B4B-PH-K-S(LF)(SN), J3 B3B-PH-K-S(LF)(SN), J4 B2B-PH-K-S(LF)(SN), J6 ESP Header, U1 LMR38020SDDAR, U2 LM66100DCKR, U3 TPS2553DBVR, U4 ADS1115IDGS, U6 TMP1075DGK

Commit message: Current
Parts:
- J1, J2: value B4B-PH-K-S(LF)(SN) -> B04B-XASK-1(LF)(SN); footprint Connector_JST:JST_PH_B4B-PH-K_1x04_P2.00mm_Vertical -> Connector_JST:JST_XA_B04B-XASK-1_1x04_P2.50mm_Vertical
- J3: value B3B-PH-K-S(LF)(SN) -> B03B-XASK-1(LF)(SN); footprint Connector_JST:JST_PH_B3B-PH-K_1x03_P2.00mm_Vertical -> Connector_JST:JST_XA_B03B-XASK-1_1x03_P2.50mm_Vertical
- J4: value B2B-PH-K-S(LF)(SN) -> B02B-XASK-1(LF)(SN); footprint Connector_JST:JST_PH_B2B-PH-K_1x02_P2.00mm_Vertical -> Connector_JST:JST_XA_B02B-XASK-1_1x02_P2.50mm_Vertical
- moved R9 12.7 mm to (183.2, 106.9), turned to 0 degrees
- moved C12 6.93 mm to (177.0, 106.8)
- moved J3 5.10 mm to (185.0, 92.0), turned to 180 degrees
- moved C18 4.73 mm to (150.2, 106.0)
- moved R8 4.51 mm to (182.3, 86.8), turned to 0 degrees
- moved R10 2.56 mm to (183.2, 104.8)
- moved C11 2.33 mm to (168.8, 91.6)
- moved D1 1.71 mm to (160.2, 91.5)
- moved D2 1.40 mm to (164.4, 91.4)
- moved R1 1.36 mm to (167.3, 88.0)
- moved J2 1.36 mm to (154.6, 92.2)
- moved TH1 1.30 mm to (159.8, 98.5)
- moved C9 1.21 mm to (170.2, 86.0), turned to 180 degrees
- moved J4 1.20 mm to (184.4, 99.8)
- moved J1 1.19 mm to (154.6, 100.0)
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Routing:
- net GND: track 0.65 -> 27.8 mm, vias 0 -> 14
- net Net-(J1-Pin_2): track 14.8 -> 32.5 mm
- net /+5V: track 69.6 -> 59.6 mm, vias 0 -> 2
- net Net-(R10-Pad1): track 12.0 -> 20.9 mm
- net Net-(J3-Pin_2): track 10.3 -> 14.7 mm
- net /+3V3: track 80.3 -> 84.1 mm
- net /+5V_SNS: track 12.0 -> 15.5 mm
- net /IGN: track 22.9 -> 19.7 mm
- net Net-(U1-RT/SYNC): track 8.39 -> 9.89 mm
- net Net-(U4-AIN0): track 34.7 -> 36.2 mm
- net /TC+: track 7.91 -> 9.24 mm
- net Net-(J1-Pin_3): track 6.55 -> 7.80 mm
- net Net-(J1-Pin_1): track 6.55 -> 7.80 mm
- net /+5V_ESP: track 12.4 -> 13.6 mm
- net /VIN_P: track 21.1 -> 22.1 mm
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Other:
- board size 46 x 46 mm -> 45 x 45 mm
