File: pcb/map-and-egt-daughterboard/map-and-egt-daughterboard.kicad_sch (KiCad schematic)
At the start: 8 parts, among them J1 Power Connector 1, J2 Power Connector 2, U1 LMR38020SDDAR

Commit message: Changes
Parts:
- added C10, C7: 1uF, Capacitor_SMD:C_0805_2012Metric, symbol Device:C
- added C11, C12, C13: 10nF, Capacitor_SMD:C_0603_1608Metric, symbol Device:C
- added C14, C17: 10nF, Capacitor_SMD:C_0805_2012Metric, symbol Device:C
- added C16, C18, C9: 100nF, Capacitor_SMD:C_0805_2012Metric, symbol Device:C
- added C3: 16V 100nF, Capacitor_SMD:C_0805_2012Metric, symbol Device:C
- added C4, C5, C6: 16V 22uF, Capacitor_SMD:C_0805_2012Metric, symbol Device:C
- added D3, D4, D5: BAV99, Package_TO_SOT_SMD:SOT-23, symbol Diode:BAV99
- added H1, H2, H3: MountingHole, MountingHole:MountingHole_2.2mm_M2, symbol Mechanical:MountingHole
- added J3: B3B-PH-K-S(LF)(SN), Connector_JST:JST_PH_B3B-PH-K_1x03_P2.00mm_Vertical, symbol Connector_Generic:Conn_01x03
- added J4: B2B-PH-K-S(LF)(SN), Connector_JST:JST_PH_B2B-PH-K_1x02_P2.00mm_Vertical, symbol Connector_Generic:Conn_01x02
- added J6: ESP Header, Connector_PinHeader_2.54mm:PinHeader_1x08_P2.54mm_Vertical, symbol Connector:Conn_01x08_Pin
- added L1: SRP7028A-150M, Inductor_SMD:L_Bourns_SRP7028A_7.3x6.6mm, symbol Device:L
- added R1: 68k, Resistor_SMD:R_0805_2012Metric, symbol Device:R
- added R10, R13, R17, R7: 1k, Resistor_SMD:R_0805_2012Metric, symbol Device:R
- added R11: 100k, Resistor_SMD:R_0805_2012Metric, symbol Device:R
- added R12: 20k, Resistor_SMD:R_0805_2012Metric, symbol Device:R
- added R14, R15: 4.7k, Resistor_SMD:R_0805_2012Metric, symbol Device:R
- added R16, R5, R6, R8, R9: 10k, Resistor_SMD:R_0805_2012Metric, symbol Device:R
- added R18: 1M, Resistor_SMD:R_0805_2012Metric, symbol Device:R
- added R2: 33k, Resistor_SMD:R_0805_2012Metric, symbol Device:R
- added R3: 8.2k, Resistor_SMD:R_0805_2012Metric, symbol Device:R
- added R4: 220k, Resistor_SMD:R_0805_2012Metric, symbol Device:R
- added U2: LM66100DCKR, Package_TO_SOT_SMD:SOT-363_SC-70-6, symbol Power_Management:LM66100DCK
- added U3: TPS2553DBVR, Package_TO_SOT_SMD:SOT-23-6, symbol Project Lib:TPS2553DBVR
- added U4: ADS1115IDGS, Package_SO:TSSOP-10_3x3mm_P0.5mm, symbol Analog_ADC:ADS1115IDGS
- added U6: TMP1075DGK, Package_SO:VSSOP-8_3x3mm_P0.65mm, symbol Sensor_Temperature:TMP1075DGK
- C1: value 4.7uF -> 50V 10uF; footprint Capacitor_SMD:C_1210_3225Metric -> Capacitor_SMD:C_0805_2012Metric; LCSC (none) -> C440198
- C2: value 0.1uF -> 100V 100nF; footprint Capacitor_SMD:C_1210_3225Metric -> Capacitor_SMD:C_0805_2012Metric; LCSC (none) -> C28233
- D1: value D_TVS -> SMBJ24CA; LCSC (none) -> C78416
- D2: value SS26 -> SS210; symbol Diode:SS26 -> Diode:SS210; LCSC (none) -> C14996
- J1: value Power Connector 1 -> B4B-PH-K-S(LF)(SN); LCSC (none) -> C131334; now left out of the parts list
- J2: value Power Connector 2 -> B4B-PH-K-S(LF)(SN); LCSC (none) -> C131334; now left out of the parts list
- TH1: value PTC -> BSMD1812-150-33V; LCSC (none) -> C883154
- U1: footprint Package_SO:SOIC-8-1EP_3.9x4.9mm_P1.27mm_EP2.95x4.9mm -> Package_SO:Texas_HSOP-8-1EP_3.9x4.9mm_P1.27mm; LCSC (none) -> C3192337
Connections:
- net at J1.1 (Pin_1): now also J2.1 (Pin_1)
- net at J1.2 (Pin_2): now also J2.2 (Pin_2), TH1.2
- net at J1.3 (Pin_3): now also J2.3 (Pin_3)
- net GND: now reaches J1.4 (Pin_4)
- net GND: now also C1.2, C2.2, D1.1 (A1), J2.4 (Pin_4), U1.1 (GND), U1.9 (EP), C10.2, C11.2, C12.2, C13.2, C14.2, C16.2, C17.2, C18.2, C4.2, C5.2, C6.2, C7.2, C9.2, D3.1 (K), D4.1 (K), D5.1 (K), J3.1 (Pin_1), J4.1 (Pin_1), J6.2 (Pin_2), R1.2, R12.1, R3.2, R4.2, R6.1, R9.1, U2.2 (GND), U2.5 (ST), U3.2 (GND), U4.1 (ADDR), U4.3 (GND), U6.4 (GND), U6.5 (A2), U6.6 (A1)
- net VIN_P: now reaches C2.1
- net VIN_P: now also C1.1, D2.1 (K), U1.2 (EN), U1.3 (VIN)
- net IGN: now reaches TH1.1
- net IGN: now also D1.2 (A2), D2.2 (A), R11.1
- net at U1.4 (RT/SYNC): now also R1.1
- net at U1.5 (FB): now also R2.2, R3.1
- net at U1.7 (BOOT): now also C3.2
- net SW: now reaches U1.8 (SW)
- net SW: now also C3.1, L1.1
- new net: C11.1, D3.3 (K), R7.2, U4.4 (AIN0)
- new net: C12.1, D4.3 (K), R10.2, U4.5 (AIN1)
- new net: R11.2, R12.2, R13.1
- new net: J3.2 (Pin_2), R5.1
- new net: R5.2, R6.2, R7.1
- new net: C13.1, D5.3 (K), R13.2, U4.6 (AIN2)
- new net: R10.1, R8.2, R9.2
- new net: R4.1, U3.5 (ILIM)
- new net +3V3: C16.1, C18.1, D3.2 (A), D4.2 (A), D5.2 (A), J6.3 (Pin_3), R14.1, R15.1, R16.1, R18.1, U4.8 (VDD), U6.7 (A0), U6.8 (V+)
- new net +5V: C4.1, C5.1, C6.1, C9.1, L1.2, R2.1, U2.1 (VIN), U3.1 (IN), U3.3 (EN)
- new net +5V_ESP: C7.1, J6.1 (Pin_1), U2.3 (~{CE}), U2.6 (VOUT)
- new net +5V_SNS: C10.1, J3.3 (Pin_3), R8.1, U3.6 (OUT)
- new net ALERT: J6.8 (Pin_8), R16.2, U4.2 (ALERT/RDY)
- new net SCL: J6.7 (Pin_7), R15.2, U4.10 (SCL), U6.2 (SCL)
- new net SDA: J6.6 (Pin_6), R14.2, U4.9 (SDA), U6.1 (SDA)
- new net TC+: C14.1, J4.2 (Pin_2), R17.1, R18.2
- new net TC_IN: C17.1, R17.2, U4.7 (AIN3)
- no-connect marks 0 -> 5
Other:
- note added: "Boost Sensor"
- note added: "ESP Header and Pullups"
- note added: "Power (12V to 5V, Protection)"
- moved on the sheet: C1, C2, D1, D2, J1, J2, TH1, U1

Commit message: Current
Parts:
- J1, J2: value B4B-PH-K-S(LF)(SN) -> B04B-XASK-1(LF)(SN); footprint Connector_JST:JST_PH_B4B-PH-K_1x04_P2.00mm_Vertical -> Connector_JST:JST_XA_B04B-XASK-1_1x04_P2.50mm_Vertical; LCSC C131334 -> C264994
- J3: value B3B-PH-K-S(LF)(SN) -> B03B-XASK-1(LF)(SN); footprint Connector_JST:JST_PH_B3B-PH-K_1x03_P2.00mm_Vertical -> Connector_JST:JST_XA_B03B-XASK-1_1x03_P2.50mm_Vertical; LCSC C131339 -> C265055
- J4: value B2B-PH-K-S(LF)(SN) -> B02B-XASK-1(LF)(SN); footprint Connector_JST:JST_PH_B2B-PH-K_1x02_P2.00mm_Vertical -> Connector_JST:JST_XA_B02B-XASK-1_1x02_P2.50mm_Vertical; LCSC C131337 -> C263753
Changed lines of the file:
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@@
 			)
 		)
-		(property "Value" "B3B-PH-K-S(LF)(SN)"
+		(property "Value" "B03B-XASK-1(LF)(SN)"
 			(at 25.4 99.06 0)
 			(show_name no)
@@
 			)
 		)
-		(property "Footprint" "Connector_JST:JST_PH_B3B-PH-K_1x03_P2.00mm_Vertical"
+		(property "Footprint" "Connector_JST:JST_XA_B03B-XASK-1_1x03_P2.50mm_Vertical"
 			(at 25.4 105.41 0)
 			(hide yes)
@@
 			)
 		)
-		(property "LCSC" "C131339"
+		(property "LCSC" "C265055"
 			(at 25.4 105.41 0)
 			(hide yes)
@@
 			)
 		)
-		(property "Value" "B4B-PH-K-S(LF)(SN)"
+		(property "Value" "B04B-XASK-1(LF)(SN)"
 			(at 41.91 50.7999 0)
 			(show_name no)
@@
 			)
 		)
-		(property "Footprint" "Connector_JST:JST_PH_B4B-PH-K_1x04_P2.00mm_Vertical"
+		(property "Footprint" "Connector_JST:JST_XA_B04B-XASK-1_1x04_P2.50mm_Vertical"
 			(at 39.37 48.26 0)
 			(hide yes)
@@
 			)
 		)
-		(property "LCSC" "C131334"
+		(property "LCSC" "C264994"
 			(at 39.37 48.26 0)
 			(hide yes)
@@
 			)
 		)
-		(property "Value" "B2B-PH-K-S(LF)(SN)"
+		(property "Value" "B02B-XASK-1(LF)(SN)"
 			(at 26.67 163.83 0)
 			(show_name no)
@@
 			)
 		)
-		(property "Footprint" "Connector_JST:JST_PH_B2B-PH-K_1x02_P2.00mm_Vertical"
+		(property "Footprint" "Connector_JST:JST_XA_B02B-XASK-1_1x02_P2.50mm_Vertical"
 			(at 26.67 170.18 0)
 			(hide yes)
@@
 			)
 		)
-		(property "LCSC" "C131337"
+		(property "LCSC" "C263753"
 			(at 26.67 170.18 0)
 			(hide yes)
@@
 			)
 		)
-		(property "Value" "B4B-PH-K-S(LF)(SN)"
+		(property "Value" "B04B-XASK-1(LF)(SN)"
 			(at 73.66 50.7999 0)
 			(show_name no)
@@
 			)
 		)
-		(property "Footprint" "Connector_JST:JST_PH_B4B-PH-K_1x04_P2.00mm_Vertical"
+		(property "Footprint" "Connector_JST:JST_XA_B04B-XASK-1_1x04_P2.50mm_Vertical"
 			(at 71.12 48.26 0)
 			(hide yes)
@@
 			)
 		)
-		(property "LCSC" "C131334"
+		(property "LCSC" "C264994"
 			(at 71.12 48.26 0)
 			(hide yes)
